File: kicad/ER1/DetecteurPresence/DetecteurPresence.sch (KiCad schematic (older format))
At the start: 41 parts, among them J1 Bornier 3 pts, J2 Bornier 2 pts, U1 TL082, U2 NE555D, U3 LM311

Commit message: Fin du projet de modelisation de circuit imprime.
Parts:
- removed R11: 10k, symbol Device:R_US
- added RV1: 10k, Potentiometer_SMD:Potentiometer_Bourns_TC33X_Vertical, symbol Device:R_POT_US
- added TP7: Vref, TestPoint:TestPoint_Bridge_Pitch2.54mm_Drill0.7mm, symbol Connector:TestPoint
- added TP8: GND, TestPoint:TestPoint_Bridge_Pitch2.54mm_Drill0.7mm, symbol Connector:TestPoint
- C1, C10, C11, C12, C4, C5, C6, C7, C8, C9: footprint (none) -> Capacitor_SMD:C_0805_2012Metric_Pad1.18x1.45mm_HandSolder
- C2, C3: footprint (none) -> Capacitor_THT:CP_Radial_D5.0mm_P2.00mm
- D3: footprint (none) -> LED_THT:LED_D5.0mm
- D4: footprint (none) -> LED_THT:LED_D5.0mm_Clear
- J1: footprint (none) -> MesEmpreintes:Bornier_3points_L15mm_W7.5mm_P5mm; Spice_Model (none) -> Alimentation; Spice_Netlist_Enabled (none) -> Y; Spice_Primitive (none) -> X
- J2: footprint (none) -> MesEmpreintes:Bornier_2points_L10mm_W7.5mm_P5mm
- L1: footprint (none) -> Inductor_THT:L_Radial_D7.5mm_P5.00mm_Fastron_07P
- R1, R10, R12, R13, R2, R3, R4, R5, R6, R8, R9: footprint (none) -> Resistor_SMD:R_0805_2012Metric_Pad1.20x1.40mm_HandSolder
- R7: value 6k8 -> 1k; footprint (none) -> Resistor_SMD:R_0805_2012Metric_Pad1.20x1.40mm_HandSolder
- TP1, TP2, TP3, TP4, TP5, TP6: footprint (none) -> TestPoint:TestPoint_Bridge_Pitch2.54mm_Drill0.7mm
- U1, U3: footprint (none) -> Package_SO:SOIC-8_3.9x4.9mm_P1.27mm
Connections:
- net GND: now also TP8.1
- net VEE: no longer R12.1
- net at R10.2, U2.7 (DIS): now also RV1.1
- net Viucr: now reaches C1.2, D1.1 (K), R1.2, U1.2 (-)
- net Vacr: now reaches R3.1, R4.2, U1.6 (-)
- net Vref: now reaches R6.2, R7.1, U3.3 (-)
- net Vref: now also TP7.1
- new net: R12.1, RV1.2, RV1.3
Other:
- note added: "* Modèle pour U1B\nXU1B /Vr /Vacr VCC VEE /Va TL082"
- note added: "* Transcaonductance Emission Réception IR\nG1 / Viucr VEE / Vast GND 0.000002"
- note removed: "* Transcaonductance Emission Réception IR\nG1 / Viucr GND / Vast GND 0.0000001"
- moved on the sheet: D4, R13, TP6
